File: receiver/GX3500-LVDS-Receiver.sch (KiCad schematic (older format))
At the start: 50 parts, among them J1 RJ45_LEDS_SHIELDED, P1 BNC, P2 BNC, P3 BNC, P4 BNC, P5 USB_B, SW1 Switch_SPDT_Shielded, U2 SN74LV125A, U3 ADum5404CRWZ, U4 SN65LVDS048A, U5 LD1117S33CTR, U6 LM393

Commit message: try to remove other unnecessary libraries
Parts:
- removed W1, W2: TEST, Measurement_Points:Test_Point_2Pads, symbol TEST-RESCUE-GX3500-LVDS-Receiver
- added W1, W2: TEST, Measurement_Points:Test_Point_2Pads, symbol TEST_2P
- P5: symbol USB_B-RESCUE-GX3500-LVDS-Receiver -> USB_B
Connections:
- net +3.3VP: now also W2.1
- net GND: now also W1.2
- net GNDREF: now also W2.2
- net VDD: now also W1.1
- no-connect marks 1 -> 4
